File: IRsensormodule.kicad_sch (KiCad schematic)
At the start: 2 parts, among them J1 Conn_01x03_Pin, J2 Conn_01x03_Pin

Commit message: V0.1 voor review
Parts:
- added C1: 0805,100nF,50V,X7R, Capacitor_SMD:C_0805_2012Metric, symbol t_jlcpcb-basic-capacitor:0805,100nF,50V,X7R
- added J10, J11, J6, J7, J8, J9: Conn_01x04_Socket, Connector_PinHeader_2.54mm:PinHeader_1x04_P2.54mm_Vertical, symbol Connector:Conn_01x04_Socket
- added J12, J13: Conn_01x01_Socket, Connector_PinSocket_2.54mm:PinSocket_1x01_P2.54mm_Vertical, symbol Connector:Conn_01x01_Socket
- added J14, J3: Conn_01x03_Socket, Connector_PinSocket_2.54mm:PinSocket_1x03_P2.54mm_Vertical, symbol Connector:Conn_01x03_Socket
- added J4: Conn_01x02_Socket, Connector_JST:JST_GH_BM02B-GHS-TBT_1x02-1MP_P1.25mm_Vertical, symbol Connector:Conn_01x02_Socket
- added J5: Conn_01x03_Socket, Connector_JST:JST_GH_BM03B-GHS-TBT_1x03-1MP_P1.25mm_Vertical, symbol Connector:Conn_01x03_Socket
- added Q1: 2N3904, Package_TO_SOT_THT:TO-92_Inline, symbol Transistor_BJT:2N3904
- added R1: 0805,10k, Resistor_SMD:R_0805_2012Metric, symbol t_jlcpcb-basic-resistor:0805,10k
- added R2: 0805,1.2k, Resistor_SMD:R_0805_2012Metric, symbol t_jlcpcb-basic-resistor:0805,1.2k
- added R3: 0805,220, Resistor_SMD:R_0805_2012Metric, symbol t_jlcpcb-basic-resistor:0805,220
- added U5: ATtiny1614-SS, Package_SO:SOIC-14_3.9x8.7mm_P1.27mm, symbol MCU_Microchip_ATtiny:ATtiny1614-SS
- J1, J2: footprint (none) -> Connector_PinHeader_2.54mm:PinHeader_1x03_P2.54mm_Vertical
Connections:
- net GND: now reaches J1.1 (Pin_1)
- net GND: now also C1.2, J3.3 (Pin_3), Q1.1 (E), U5.14 (GND)
- net VBAT: now reaches J1.2 (Pin_2)
- net +3V3: now reaches J1.3 (Pin_3)
- net +3V3: now also C1.1, J12.1 (Pin_1), J13.1 (Pin_1), J3.1 (Pin_1), J5.3 (Pin_3), R1.1, R3.2, U5.1 (VCC)
- net SMBA: now reaches J2.1 (Pin_1)
- net SDA: now reaches J2.2 (Pin_2)
- net SDA: now also U5.8 (PB1)
- net SCL: now reaches J2.3 (Pin_3)
- net SCL: now also U5.9 (PB0)
- new net: J4.2 (Pin_2), R3.1
- new net: Q1.2 (B), R2.2
- new net IRdataIN: J5.2 (Pin_2), R1.2, U5.5 (PA7)
- new net IRledcontrol: R2.1, U5.4 (PA6)
- new net PA1: J7.3 (Pin_3), U5.11 (PA1)
- new net PA2: J7.2 (Pin_2), U5.12 (PA2)
- new net PA3: J7.1 (Pin_1), U5.13 (PA3)
- new net PA4: J6.4 (Pin_4), U5.2 (PA4)
- new net PA5: J6.3 (Pin_3), U5.3 (PA5)
- new net PB2: J6.2 (Pin_2), U5.7 (PB2)
- new net PB3: J6.1 (Pin_1), U5.6 (PB3)
- new net UPDI: J3.2 (Pin_2), U5.10 (~{RESET}/PA0)
- new net emitreceive: J4.1 (Pin_1), J5.1 (Pin_1), Q1.3 (C)
- no-connect marks 0 -> 20
Other:
- note added: "3V3 external prototyping points"
- note added: "ATtiny pins"
- note added: "Attiny1614-ss"
- note added: "Prototyping holes"
- note added: "Switching Transistor"
- note added: "UDPI connector"
- note removed: "Data -> I2C"
- note removed: "Data logic(driver chips/levelshifter)"
